File: hardware/Detector/chamber.kicad_pcb (KiCad board)
At the start: 2 copper layers, 100 x 100 mm, 93 parts, among them J1 USB_B_Micro, J31 Conn_01x04_Female, J32 Conn_01x04_Female, J33 Conn_01x04_Male, J34 Conn_01x04_Male, J35 Conn_01x04_Female, J36 Conn_01x04_Female, J37 Conn_01x04_Male, J38 Conn_01x04_Male, J51 Conn_02x05_Counter_Clockwise, J52 Conn_01x04, Q31 BC859, Q32 Q_NMOS_GDS, U1 STM32F030K6Tx, U21 LM324, U31 MC34063AD, U54 STM8S003F3P

Commit message: backup copy
Parts:
- removed J31, J32, J35, J36: Conn_01x04_Female, Connector_PinSocket_2.54mm:PinSocket_1x04_P2.54mm_Vertical_SMD_Pin1Right
- removed J33, J34, J37, J38: Conn_01x04_Male, Connector_PinHeader_2.54mm:PinHeader_1x04_P2.54mm_Vertical_SMD_Pin1Right
- removed R22, R24, R25, R26, R27, R28, R29, R30, R38, R40, R41, R42, R45, R46: R, Resistor_SMD:R_0805_2012Metric_Pad1.15x1.40mm_HandSolder
- removed RV21: R_POT_TRIM, Potentiometer_THT:Potentiometer_Bourns_3296W_Vertical
- removed U21: LM324, Package_SO:SOIC-14_3.9x8.7mm_P1.27mm
- added D2: D_Zener, Diode_SMD:D_MiniMELF, F.Cu at (178.5, 112.5)
- added D3: D_Zener, Diode_SMD:D_MiniMELF, F.Cu at (178.5, 115.8)
- added D4: D_Zener, Diode_SMD:D_MiniMELF, F.Cu at (188.8, 112.5)
- added D5: D_Zener, Diode_SMD:D_MiniMELF, F.Cu at (178.5, 119.0)
- added J10: Conn_02x02_Odd_Even, Connector_PinSocket_2.54mm:PinSocket_2x02_P2.54mm_Vertical_SMD, F.Cu at (182.5, 98.7)
- added J11: Conn_02x02_Odd_Even, Connector_PinHeader_2.54mm:PinHeader_2x02_P2.54mm_Vertical_SMD, F.Cu at (170.0, 90.5)
- added J12: Conn_02x02_Odd_Even, Connector_PinSocket_2.54mm:PinSocket_2x02_P2.54mm_Vertical_SMD, F.Cu at (192.6, 91.5)
- added J13: Conn_02x02_Odd_Even, Connector_PinHeader_2.54mm:PinHeader_2x02_P2.54mm_Vertical_SMD, F.Cu at (158.2, 105.8)
- added J14: Conn_02x02_Odd_Even, Connector_PinSocket_2.54mm:PinSocket_2x02_P2.54mm_Vertical_SMD, F.Cu at (179.8, 105.8)
- added J15: Conn_02x02_Odd_Even, Connector_PinHeader_2.54mm:PinHeader_2x02_P2.54mm_Vertical_SMD, F.Cu at (171.0, 98.7)
- added J2: Conn_02x02_Odd_Even, Connector_PinSocket_2.54mm:PinSocket_2x02_P2.54mm_Vertical_SMD, B.Cu at (125.0, 76.0)
- added J3: Conn_02x02_Odd_Even, Connector_PinHeader_2.54mm:PinHeader_2x02_P2.54mm_Vertical_SMD, F.Cu at (125.0, 76.0)
- added J4: Conn_02x02_Odd_Even, Connector_PinSocket_2.54mm:PinSocket_2x02_P2.54mm_Vertical_SMD, B.Cu at (125.0, 83.0)
- added J5: Conn_02x02_Odd_Even, Connector_PinHeader_2.54mm:PinHeader_2x02_P2.54mm_Vertical_SMD, F.Cu at (125.0, 83.2)
- added J6: Conn_02x02_Odd_Even, Connector_PinSocket_2.54mm:PinSocket_2x02_P2.54mm_Vertical_SMD, F.Cu at (182.5, 91.5)
- added J7: Conn_02x02_Odd_Even, Connector_PinHeader_2.54mm:PinHeader_2x02_P2.54mm_Vertical_SMD, F.Cu at (158.2, 91.5)
- added J8: Conn_02x02_Odd_Even, Connector_PinHeader_2.54mm:PinHeader_2x02_P2.54mm_Vertical_SMD, F.Cu at (158.2, 98.7)
- added J9: Conn_02x02_Odd_Even, Connector_PinSocket_2.54mm:PinSocket_2x02_P2.54mm_Vertical_SMD, F.Cu at (169.7, 105.8)
- added U2: 74LS14, Package_SO:SOIC-14_3.9x8.7mm_P1.27mm, F.Cu at (187.9, 119.2)
- C41, C43: footprint Capacitor_THT:C_Disc_D8.0mm_W2.5mm_P5.00mm -> Capacitor_THT:C_Rect_L19.0mm_W7.0mm_P15.00mm_MKS4
- moved C32 94.8 mm to (128.1, 149.5), turned to 270 degrees
- moved U31 82.6 mm to (127.5, 143.3), turned to 90 degrees
- moved C31 78.9 mm to (131.6, 141.9), turned to 270 degrees
- moved R35 71.0 mm to (125.0, 136.8), turned to 270 degrees
- moved R32 68.9 mm to (130.7, 136.8), turned to 0 degrees
- moved C35 66.3 mm to (149.6, 131.9), turned to 270 degrees
- moved R34 64.6 mm to (126.0, 133.7), turned to 180 degrees
- moved C2 63.6 mm to (146.4, 131.9), turned to 270 degrees
- moved Q31 61.9 mm to (130.8, 133.3), turned to 90 degrees
- moved C39 59.6 mm to (126.1, 131.2), turned to 180 degrees
- moved Q32 57.8 mm to (140.8, 130.7), turned to 180 degrees
- moved D32 53.8 mm to (130.8, 129.2), turned to 90 degrees
- moved R31 52.9 mm to (143.9, 127.1), turned to 90 degrees
- moved L31 45.3 mm to (140.2, 124.4), turned to 180 degrees
- moved H3 37.4 mm to (119.0, 92.5)
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Connections:
- R47 pad 1: Net-(J31-Pad1) -> (no net)
- R48 pad 1: Net-(J31-Pad2) -> (no net)
- R49 pad 1: Net-(J31-Pad3) -> (no net)
- R50 pad 1: Net-(J31-Pad4) -> (no net)
- R51 pad 1: Net-(J32-Pad1) -> (no net)
- R52 pad 1: Net-(J32-Pad2) -> (no net)
- R53 pad 1: Net-(J32-Pad3) -> (no net)
- R54 pad 1: Net-(J32-Pad4) -> (no net)
- R65 pad 1: Net-(J35-Pad1) -> (no net)
- R66 pad 1: Net-(J35-Pad2) -> (no net)
- R67 pad 1: Net-(J35-Pad3) -> (no net)
- R68 pad 1: Net-(J35-Pad4) -> (no net)
- R69 pad 1: Net-(J36-Pad1) -> (no net)
- R70 pad 1: Net-(J36-Pad2) -> (no net)
- R71 pad 1: Net-(J36-Pad3) -> (no net)
- R72 pad 1: Net-(J36-Pad4) -> (no net)
Routing:
- net INT2: track 90.8 -> 0.00 mm
- net INT1: track 50.8 -> 0.00 mm
- net Net-(C25-Pad1): track 37.8 -> 9.20 mm
- net INT3: track 26.8 -> 0.00 mm
- net Net-(C22-Pad1): track 34.5 -> 14.5 mm
- net Net-(C21-Pad1): track 36.9 -> 17.5 mm, vias 2 -> 1
- net INT4: track 19.1 -> 0.00 mm
- net VCC_5V: track 136.0 -> 117.2 mm, vias 6 -> 4
- net Net-(C24-Pad1): track 28.7 -> 13.8 mm
- net Net-(R27-Pad2): track 12.2 -> 0.00 mm
- net Net-(R27-Pad1): track 5.57 -> 0.00 mm
- net Net-(R42-Pad1): track 5.32 -> 0.00 mm
- net Net-(R28-Pad1): track 5.17 -> 0.00 mm
- net Net-(R41-Pad1): track 5.15 -> 0.00 mm
- net Net-(C39-Pad1): track 33.0 -> 35.9 mm
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
Commit message: backup
Parts:
- removed R47, R48, R50, R51, R52, R53, R54, R65, R66, R67, R68, R69, R70, R71, R72: R, Resistor_SMD:R_0805_2012Metric_Pad1.15x1.40mm_HandSolder
- added R10: R, Resistor_SMD:R_0805_2012Metric_Pad1.15x1.40mm_HandSolder, F.Cu at (158.6, 118.9)
- added R11: R, Resistor_SMD:R_0805_2012Metric_Pad1.15x1.40mm_HandSolder, F.Cu at (174.9, 121.9)
- added R12: R, Resistor_SMD:R_0805_2012Metric_Pad1.15x1.40mm_HandSolder, F.Cu at (158.6, 121.4)
- added R13: R, Resistor_SMD:R_0805_2012Metric_Pad1.15x1.40mm_HandSolder, F.Cu at (174.9, 132.1)
- added R14: R, Resistor_SMD:R_0805_2012Metric_Pad1.15x1.40mm_HandSolder, F.Cu at (158.6, 132.1)
- added R15: R, Resistor_SMD:R_0805_2012Metric_Pad1.15x1.40mm_HandSolder, F.Cu at (174.9, 134.6)
- added R16: R, Resistor_SMD:R_0805_2012Metric_Pad1.15x1.40mm_HandSolder, F.Cu at (158.6, 134.6)
- added R2: R, Resistor_SMD:R_0805_2012Metric_Pad1.15x1.40mm_HandSolder, F.Cu at (158.7, 126.0)
- added R3: R, Resistor_SMD:R_0805_2012Metric_Pad1.15x1.40mm_HandSolder, F.Cu at (174.9, 128.5)
- added R4: R, Resistor_SMD:R_0805_2012Metric_Pad1.15x1.40mm_HandSolder, F.Cu at (158.7, 128.6)
- added R5: R, Resistor_SMD:R_0805_2012Metric_Pad1.15x1.40mm_HandSolder, F.Cu at (174.9, 112.3)
- added R6: R, Resistor_SMD:R_0805_2012Metric_Pad1.15x1.40mm_HandSolder, F.Cu at (158.6, 112.3)
- added R7: R, Resistor_SMD:R_0805_2012Metric_Pad1.15x1.40mm_HandSolder, F.Cu at (174.9, 115.1)
- added R8: R, Resistor_SMD:R_0805_2012Metric_Pad1.15x1.40mm_HandSolder, F.Cu at (158.6, 114.8)
- added R9: R, Resistor_SMD:R_0805_2012Metric_Pad1.15x1.40mm_HandSolder, F.Cu at (174.9, 118.9)
- C41, C43: footprint Capacitor_THT:C_Rect_L19.0mm_W7.0mm_P15.00mm_MKS4 -> Capacitor_THT:C_Rect_L13.0mm_W8.0mm_P10.00mm_FKS3_FKP3_MKS4
- J10, J12, J14, J6: moved to B.Cu
- J8: footprint Connector_PinHeader_2.54mm:PinHeader_2x02_P2.54mm_Vertical_SMD -> Connector_PinSocket_2.54mm:PinSocket_2x02_P2.54mm_Vertical_SMD; moved to B.Cu
- J9: footprint Connector_PinSocket_2.54mm:PinSocket_2x02_P2.54mm_Vertical_SMD -> Connector_PinHeader_2.54mm:PinHeader_2x02_P2.54mm_Vertical_SMD
- moved J12 49.4 mm to (166.8, 133.6), turned to 180 degrees
- moved J6 38.8 mm to (166.8, 127.0), turned to 180 degrees
- moved J7 36.5 mm to (166.8, 127.0)
- moved C23 30.3 mm to (179.2, 95.2)
- moved J11 30.1 mm to (166.8, 120.4)
- moved J13 29.1 mm to (166.8, 133.6)
- moved J10 26.8 mm to (166.8, 120.4), turned to 180 degrees
- moved D2 21.6 mm to (186.0, 132.8), turned to 90 degrees
- moved C41 21.3 mm to (134.1, 95.0), turned to 0 degrees
- moved U2 20.7 mm to (177.4, 101.5)
- moved R21 20.1 mm to (120.9, 125.0), turned to 270 degrees
- moved R49 20.0 mm to (174.9, 126.0), turned to 0 degrees
- moved J8 17.4 mm to (166.8, 113.8), turned to 180 degrees
- moved D5 17.1 mm to (185.8, 103.5), turned to 270 degrees
- moved R39 15.7 mm to (128.0, 97.5), turned to 180 degrees
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Connections:
- J10 pad 1: (no net) -> Net-(J10-Pad1)
- J10 pad 2: (no net) -> Net-(J10-Pad2)
- J10 pad 3: (no net) -> Net-(J10-Pad3)
- J10 pad 4: (no net) -> Net-(J10-Pad4)
- J11 pad 1: (no net) -> Net-(J10-Pad1)
- J11 pad 2: (no net) -> Net-(J10-Pad2)
- J11 pad 3: (no net) -> Net-(J10-Pad3)
- J11 pad 4: (no net) -> Net-(J10-Pad4)
- J12 pad 1: (no net) -> Net-(J12-Pad1)
- J12 pad 2: (no net) -> Net-(J12-Pad2)
- J12 pad 3: (no net) -> Net-(J12-Pad3)
- J12 pad 4: (no net) -> Net-(J12-Pad4)
- J13 pad 1: (no net) -> Net-(J12-Pad1)
- J13 pad 2: (no net) -> Net-(J12-Pad2)
- J13 pad 3: (no net) -> Net-(J12-Pad3)
- J13 pad 4: (no net) -> Net-(J12-Pad4)
- J14 pad 1: (no net) -> VCC_5V
- J14 pad 2: (no net) -> GND
- J14 pad 3: (no net) -> VCC_5V
- J14 pad 4: (no net) -> GND
- J15 pad 1: (no net) -> VCC_5V
- J15 pad 2: (no net) -> GND
- J15 pad 3: (no net) -> VCC_5V
- J15 pad 4: (no net) -> GND
- J6 pad 2: Net-(J6-Pad1) -> Net-(J6-Pad2)
- J6 pad 3: Net-(J6-Pad1) -> Net-(J6-Pad3)
- J6 pad 4: Net-(J6-Pad1) -> Net-(J6-Pad4)
- J7 pad 2: Net-(J6-Pad1) -> Net-(J6-Pad2)
- J7 pad 3: Net-(J6-Pad1) -> Net-(J6-Pad3)
- J7 pad 4: Net-(J6-Pad1) -> Net-(J6-Pad4)
- J8 pad 1: (no net) -> Net-(J8-Pad1)
- J8 pad 2: (no net) -> Net-(J8-Pad2)
- J8 pad 3: (no net) -> Net-(J8-Pad3)
- J8 pad 4: (no net) -> Net-(J8-Pad4)
- J9 pad 1: (no net) -> Net-(J8-Pad1)
- J9 pad 2: (no net) -> Net-(J8-Pad2)
- J9 pad 3: (no net) -> Net-(J8-Pad3)
- J9 pad 4: (no net) -> Net-(J8-Pad4)
- R49 pad 1: (no net) -> Net-(J6-Pad2)
- R49 pad 2: INT3 -> INT1
Routing:
- net INT3: track 0.00 -> 56.0 mm
- net GM_LAMP_POLARIZATION: track 30.9 -> 83.3 mm
- net INT4: track 0.00 -> 36.2 mm, vias 0 -> 4
- net INT1: track 0.00 -> 28.5 mm
- net Net-(GM1-Pad1): track 43.6 -> 17.1 mm
- net INT2: track 0.00 -> 24.5 mm, vias 0 -> 4
- net VCC_5V: track 117.2 -> 95.4 mm, vias 4 -> 3
- net Net-(GM3-Pad1): track 36.8 -> 16.8 mm
- net Net-(C24-Pad1): track 13.8 -> 33.0 mm, vias 0 -> 1
- net Net-(GM5-Pad1): track 30.1 -> 19.2 mm
- net Net-(GM7-Pad1): track 24.4 -> 13.6 mm
- net Net-(J12-Pad3): track 0.00 -> 8.25 mm, vias 0 -> 1
- net Net-(J12-Pad1): track 0.00 -> 8.25 mm, vias 0 -> 1
- net Net-(J10-Pad1): track 0.00 -> 7.93 mm, vias 0 -> 1
- net Net-(J10-Pad3): track 0.00 -> 7.93 mm, vias 0 -> 1
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Other:
- board size 100 x 100 mm -> 90 x 100 mm
- board text removed: "ADC converter"
- board text removed: "Chamber signal amplifier"
- board text removed: "analog output"

Commit message: draft
Parts:
- removed C52: 100n, Capacitor_SMD:C_0805_2012Metric_Pad1.15x1.40mm_HandSolder
- removed TP52: TestPoint, TestPoint:TestPoint_THTPad_1.0x1.0mm_Drill0.5mm
- removed U54: STM8S003F3P, Package_SO:TSSOP-20_4.4x6.5mm_P0.65mm
- moved J4 66.1 mm to (149.9, 144.3), turned to 180 degrees
- moved J5 66.0 mm to (149.9, 144.3), turned to 180 degrees
- moved U1 21.3 mm to (165.6, 72.1)
Connections:
- net INT1 renamed GM1
- net INT2 renamed GM2
- net INT3 renamed GM3
- net INT4 renamed GM4
- J10 pad 1: Net-(J10-Pad1) -> INT23
- J10 pad 2: Net-(J10-Pad2) -> INT21
- J10 pad 3: Net-(J10-Pad3) -> INT24
- J10 pad 4: Net-(J10-Pad4) -> INT22
- J11 pad 1: Net-(J10-Pad1) -> INT23
- J11 pad 2: Net-(J10-Pad2) -> INT21
- J11 pad 3: Net-(J10-Pad3) -> INT24
- J11 pad 4: Net-(J10-Pad4) -> INT22
- J12 pad 1: Net-(J12-Pad1) -> INT33
- J12 pad 2: Net-(J12-Pad2) -> INT31
- J12 pad 3: Net-(J12-Pad3) -> INT34
- J12 pad 4: Net-(J12-Pad4) -> INT32
- J13 pad 1: Net-(J12-Pad1) -> INT33
- J13 pad 2: Net-(J12-Pad2) -> INT31
- J13 pad 3: Net-(J12-Pad3) -> INT34
- J13 pad 4: Net-(J12-Pad4) -> INT32
- J51 pad 2: /DataAcquisition/SWIM -> (no net)
- J52 pad 2: /DataAcquisition/TX -> (no net)
- J52 pad 3: /DataAcquisition/RX -> (no net)
- J6 pad 1: Net-(J6-Pad1) -> INT03
- J6 pad 2: Net-(J6-Pad2) -> INT01
- J6 pad 3: Net-(J6-Pad3) -> INT04
- J6 pad 4: Net-(J6-Pad4) -> INT02
- J7 pad 1: Net-(J6-Pad1) -> INT03
- J7 pad 2: Net-(J6-Pad2) -> INT01
- J7 pad 3: Net-(J6-Pad3) -> INT04
- J7 pad 4: Net-(J6-Pad4) -> INT02
- J8 pad 1: Net-(J8-Pad1) -> INT13
- J8 pad 2: Net-(J8-Pad2) -> INT11
- J8 pad 3: Net-(J8-Pad3) -> INT14
- J8 pad 4: Net-(J8-Pad4) -> INT12
- J9 pad 1: Net-(J8-Pad1) -> INT13
- J9 pad 2: Net-(J8-Pad2) -> INT11
- J9 pad 3: Net-(J8-Pad3) -> INT14
- J9 pad 4: Net-(J8-Pad4) -> INT12
- R10 pad 2: Net-(J10-Pad1) -> INT23
- R11 pad 1: Net-(J10-Pad4) -> INT22
- R12 pad 2: Net-(J10-Pad3) -> INT24
- R13 pad 1: Net-(J12-Pad2) -> INT31
- R14 pad 2: Net-(J12-Pad1) -> INT33
- R15 pad 1: Net-(J12-Pad4) -> INT32
- R16 pad 2: Net-(J12-Pad3) -> INT34
- R2 pad 2: Net-(J6-Pad1) -> INT03
- R3 pad 1: Net-(J6-Pad4) -> INT02
- R4 pad 2: Net-(J6-Pad3) -> INT04
- R49 pad 1: Net-(J6-Pad2) -> INT01
- R5 pad 1: Net-(J8-Pad2) -> INT11
- R6 pad 2: Net-(J8-Pad1) -> INT13
- R7 pad 1: Net-(J8-Pad4) -> INT12
- R8 pad 2: Net-(J8-Pad3) -> INT14
- R9 pad 1: Net-(J10-Pad2) -> INT21
- U1 pad 10: (no net) -> INT11
- U1 pad 11: (no net) -> INT12
- U1 pad 12: (no net) -> INT13
- U1 pad 13: (no net) -> INT14
- U1 pad 18: (no net) -> INT21
- U1 pad 19: (no net) -> INT22
- U1 pad 20: (no net) -> INT23
- U1 pad 21: (no net) -> INT24
- U1 pad 22: (no net) -> INT31
- U1 pad 23: (no net) -> INT32
- U1 pad 24: (no net) -> INT33
- U1 pad 25: (no net) -> INT34
- U1 pad 6: (no net) -> INT01
- U1 pad 7: (no net) -> INT02
- U1 pad 8: (no net) -> INT03
- U1 pad 9: (no net) -> INT04
Routing:
- net /DataAcquisition/SCL: track 27.8 -> 1.09 mm, vias 2 -> 0
- net /DataAcquisition/SDA: track 29.2 -> 3.43 mm, vias 2 -> 1
- net /DataAcquisition/SWIM: track 23.7 -> 0.00 mm
- net VCC_5V: track 95.4 -> 78.5 mm, vias 3 -> 2
- net /DataAcquisition/RX: track 14.9 -> 0.00 mm, vias 1 -> 0
- net /DataAcquisition/RST: track 16.7 -> 2.59 mm
- net (no net): track 14.5 -> 24.3 mm, vias 1 -> 0
- net /DataAcquisition/TX: track 9.60 -> 0.00 mm, vias 1 -> 0
- net Net-(J12-Pad3): track 8.25 -> 0.00 mm, vias 1 -> 0
- net Net-(J12-Pad1): track 8.25 -> 0.00 mm, vias 1 -> 0
- net INT34: track 0.00 -> 8.25 mm, vias 0 -> 1
- net INT33: track 0.00 -> 8.25 mm, vias 0 -> 1
- net Net-(J10-Pad1): track 7.93 -> 0.00 mm, vias 1 -> 0
- net INT23: track 0.00 -> 7.93 mm, vias 0 -> 1
- net Net-(J10-Pad3): track 7.93 -> 0.00 mm, vias 1 -> 0
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
Commit message: backup
Parts:
- removed C53: 100n, Capacitor_SMD:C_0805_2012Metric_Pad1.15x1.40mm_HandSolder
- added D10: 1n148, Diode_SMD:D_MiniMELF, B.Cu at (176.2, 139.2)
- added D11: 1n148, Diode_SMD:D_MiniMELF, B.Cu at (176.1, 125.7)
- added D12: 1n148, Diode_SMD:D_MiniMELF, B.Cu at (176.3, 132.6)
- added D13: 1n148, Diode_SMD:D_MiniMELF, B.Cu at (176.2, 145.3)
- added D14: 1n148, Diode_SMD:D_MiniMELF, B.Cu at (158.2, 136.4)
- added D15: 1n148, Diode_SMD:D_MiniMELF, B.Cu at (158.7, 122.9)
- added D16: 1n148, Diode_SMD:D_MiniMELF, B.Cu at (158.5, 129.5)
- added D17: 1n148, Diode_SMD:D_MiniMELF, B.Cu at (158.3, 142.7)
- added D18: 1n148, Diode_SMD:D_MiniMELF, B.Cu at (158.3, 139.4)
- added D19: 1n148, Diode_SMD:D_MiniMELF, B.Cu at (158.5, 125.7)
- added D20: 1n148, Diode_SMD:D_MiniMELF, B.Cu at (158.3, 132.3)
- added D21: 1n148, Diode_SMD:D_MiniMELF, B.Cu at (158.2, 145.5)
- added D40: LED, LED_SMD:LED_0603_1608Metric, F.Cu at (128.4, 75.0)
- added D41: LED, LED_SMD:LED_0603_1608Metric, F.Cu at (132.5, 75.0)
- added D42: LED, LED_SMD:LED_0603_1608Metric, F.Cu at (136.5, 75.0)
- added D43: 1n148, Diode_SMD:D_MiniMELF, F.Cu at (166.3, 108.7)
- added D44: 1n148, Diode_SMD:D_MiniMELF, F.Cu at (163.9, 111.8)
- added D45: 1n148, Diode_SMD:D_MiniMELF, F.Cu at (170.4, 111.8)
- added D46: 1n148, Diode_SMD:D_MiniMELF, F.Cu at (159.3, 109.2)
- added D6: 1n148, Diode_SMD:D_MiniMELF, B.Cu at (176.1, 136.7)
- added D7: 1n148, Diode_SMD:D_MiniMELF, B.Cu at (176.1, 122.9)
- added D8: 1n148, Diode_SMD:D_MiniMELF, B.Cu at (176.0, 129.5)
- added D9: 1n148, Diode_SMD:D_MiniMELF, B.Cu at (176.3, 142.7)
- added J16: Conn_02x02_Odd_Even, Connector_PinSocket_2.54mm:PinSocket_2x02_P2.54mm_Vertical_SMD, B.Cu at (167.1, 117.9)
- added J17: Conn_02x02_Odd_Even, Connector_PinHeader_2.54mm:PinHeader_2x02_P2.54mm_Vertical_SMD, F.Cu at (167.1, 117.9)
- added R17: 680R, Resistor_SMD:R_0805_2012Metric_Pad1.15x1.40mm_HandSolder, F.Cu at (127.7, 74.0)
- added R18: 680R, Resistor_SMD:R_0805_2012Metric_Pad1.15x1.40mm_HandSolder, F.Cu at (158.5, 85.9)
- added R19: 680R, Resistor_SMD:R_0805_2012Metric_Pad1.15x1.40mm_HandSolder, F.Cu at (134.1, 70.5)
- added R20: R, Resistor_SMD:R_0805_2012Metric_Pad1.15x1.40mm_HandSolder, F.Cu at (161.6, 106.7)
- added R22: R, Resistor_SMD:R_0805_2012Metric_Pad1.15x1.40mm_HandSolder, F.Cu at (159.5, 119.4)
- added R24: R, Resistor_SMD:R_0805_2012Metric_Pad1.15x1.40mm_HandSolder, F.Cu at (173.7, 119.4)
- added R25: R, Resistor_SMD:R_0805_2012Metric_Pad1.15x1.40mm_HandSolder, F.Cu at (173.7, 116.8)
- added R26: R, Resistor_SMD:R_0805_2012Metric_Pad1.15x1.40mm_HandSolder, F.Cu at (159.5, 116.3)
- added R27: 680R, Resistor_SMD:R_0805_2012Metric_Pad1.15x1.40mm_HandSolder, F.Cu at (167.6, 95.5)
- added R28: 680R, Resistor_SMD:R_0805_2012Metric_Pad1.15x1.40mm_HandSolder, F.Cu at (170.7, 95.2)
- added R29: 680R, Resistor_SMD:R_0805_2012Metric_Pad1.15x1.40mm_HandSolder, F.Cu at (154.7, 95.5)
- added R30: 680R, Resistor_SMD:R_0805_2012Metric_Pad1.15x1.40mm_HandSolder, F.Cu at (151.4, 94.7)
- U2: value 74LS14 -> HEF4093B
- moved R1 39.2 mm to (127.5, 83.6), turned to 0 degrees
- moved D1 39.2 mm to (127.5, 81.1), turned to 0 degrees
- moved J1 39.2 mm to (127.5, 81.8), turned to 270 degrees
- moved H4 34.9 mm to (189.0, 89.4), turned to 90 degrees
- moved C1 33.4 mm to (131.6, 81.8), turned to 90 degrees
- moved R60 26.0 mm to (176.8, 77.3), turned to 180 degrees
- moved R59 23.0 mm to (177.7, 74.7), turned to 180 degrees
- moved J51 22.6 mm to (152.6, 71.9), turned to 0 degrees
- moved D51 18.1 mm to (175.2, 71.9), turned to 180 degrees
- moved J14 13.2 mm to (185.6, 79.0)
- moved C23 13.2 mm to (184.3, 83.0)
- moved J15 13.1 mm to (185.4, 79.0)
- moved J52 13.0 mm to (164.3, 78.0), turned to 270 degrees
- moved J6 10.7 mm to (167.3, 137.7)
- moved J7 10.7 mm to (167.3, 137.7)
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Connections:
- R59 pad 1: /DataAcquisition/SCL -> (no net)
- R60 pad 1: /DataAcquisition/SDA -> (no net)
- U1 pad 10: INT11 -> (no net)
- U1 pad 11: INT12 -> (no net)
- U1 pad 12: INT13 -> (no net)
- U1 pad 13: INT14 -> (no net)
- U1 pad 18: INT21 -> (no net)
- U1 pad 19: INT22 -> (no net)
- U1 pad 2: /DataAcquisition/SDA -> (no net)
- U1 pad 20: INT23 -> (no net)
- U1 pad 21: INT24 -> (no net)
- U1 pad 22: INT31 -> (no net)
- U1 pad 23: INT32 -> (no net)
- U1 pad 24: INT33 -> (no net)
- U1 pad 25: INT34 -> (no net)
- U1 pad 3: /DataAcquisition/SCL -> (no net)
- U1 pad 6: INT01 -> (no net)
- U1 pad 7: INT02 -> (no net)
- U1 pad 8: INT03 -> (no net)
- U1 pad 9: INT04 -> (no net)
- U2 pad 10: (no net) -> GM2
- U2 pad 11: GND -> GM4
- U2 pad 12: (no net) -> Net-(C25-Pad1)
- U2 pad 13: GND -> Net-(C25-Pad1)
- U2 pad 2: GM1 -> Net-(C21-Pad1)
- U2 pad 3: Net-(C22-Pad1) -> GM1
- U2 pad 4: GM2 -> GM3
- U2 pad 6: GM3 -> Net-(C24-Pad1)
- U2 pad 8: GM4 -> Net-(C22-Pad1)
- U2 pad 9: Net-(C25-Pad1) -> Net-(C22-Pad1)
Routing:
- net COL1: track 0.00 -> 65.9 mm, vias 0 -> 1
- net COL3: track 0.00 -> 61.8 mm, vias 0 -> 1
- net COL0: track 0.00 -> 59.9 mm, vias 0 -> 4
- net COL2: track 0.00 -> 55.8 mm, vias 0 -> 4
- net VCC_5V: track 78.5 -> 132.1 mm
- net Net-(C24-Pad1): track 33.0 -> 14.1 mm
- net GM4: track 36.2 -> 31.3 mm
- net (no net): track 24.3 -> 28.0 mm
- net /DataAcquisition/SDA: track 3.43 -> 0.00 mm, vias 1 -> 0
- net Net-(GM5-Pad1): track 19.2 -> 15.8 mm
- net GM2: track 24.5 -> 21.6 mm
- net GM_LAMP_POLARIZATION: track 83.3 -> 85.8 mm
- net GND: track 20.4 -> 17.9 mm, vias 12 -> 5
- net GM1: track 28.5 -> 26.1 mm
- net GM3: track 56.0 -> 54.1 mm
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Other:
- board size 90 x 100 mm -> 89.9 x 82.6 mm

Commit message: backup
Parts:
- moved C23 63.3 mm to (172.7, 145.3), turned to 90 degrees
- moved U2 46.6 mm to (166.6, 143.8), turned to 270 degrees
- moved R22 20.9 mm to (173.7, 104.1)
- moved R25 19.2 mm to (157.5, 106.7), turned to 180 degrees
- moved D45 17.2 mm to (161.5, 97.0)
- moved R30 16.9 mm to (166.6, 87.4)
- moved R27 14.6 mm to (153.9, 90.4)
- moved R28 14.6 mm to (157.0, 90.2)
- moved U1 13.7 mm to (173.2, 88.9)
- moved D44 13.3 mm to (170.2, 100.1), turned to 180 degrees
- moved R24 12.7 mm to (173.7, 106.7), turned to 0 degrees
- moved R26 12.4 mm to (157.5, 104.1), turned to 180 degrees
- moved D43 12.3 mm to (170.2, 97.0), turned to 180 degrees
- moved D10 12.3 mm to (174.7, 127.0)
- moved D11 12.3 mm to (174.5, 113.5)
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Connections:
- J16 pad 1: Net-(J16-Pad1) -> ROW3
- J16 pad 3: Net-(J16-Pad3) -> ROW2
- J16 pad 4: Net-(J16-Pad4) -> ROW1
- J17 pad 1: Net-(J16-Pad1) -> ROW3
- J17 pad 3: Net-(J16-Pad3) -> ROW2
- J17 pad 4: Net-(J16-Pad4) -> ROW1
- R24 pad 1: Net-(J16-Pad4) -> ROW1
- R25 pad 1: Net-(J16-Pad3) -> ROW2
- R26 pad 1: Net-(J16-Pad1) -> ROW3
- U1 pad 11: (no net) -> ROW3
- U1 pad 12: (no net) -> ROW2
- U1 pad 13: (no net) -> ROW1
- U1 pad 18: (no net) -> ROW0
- U1 pad 21: (no net) -> COL0
- U1 pad 22: (no net) -> COL1
- U1 pad 23: (no net) -> COL2
- U1 pad 24: (no net) -> COL3
- U2 pad 1: Net-(C21-Pad1) -> Net-(C24-Pad1)
- U2 pad 10: GM2 -> GM1
- U2 pad 11: GM4 -> GM2
- U2 pad 12: Net-(C25-Pad1) -> Net-(C22-Pad1)
- U2 pad 13: Net-(C25-Pad1) -> Net-(C22-Pad1)
- U2 pad 2: Net-(C21-Pad1) -> Net-(C24-Pad1)
- U2 pad 3: GM1 -> GM3
- U2 pad 4: GM3 -> GM4
- U2 pad 5: Net-(C24-Pad1) -> Net-(C25-Pad1)
- U2 pad 6: Net-(C24-Pad1) -> Net-(C25-Pad1)
- U2 pad 8: Net-(C22-Pad1) -> Net-(C21-Pad1)
- U2 pad 9: Net-(C22-Pad1) -> Net-(C21-Pad1)
Routing:
- net Net-(C25-Pad1): track 14.2 -> 70.6 mm
- net Net-(C24-Pad1): track 14.1 -> 55.1 mm
- net Net-(D43-Pad2): track 0.00 -> 40.6 mm
- net Net-(C22-Pad1): track 14.1 -> 54.4 mm
- net Net-(C21-Pad1): track 13.6 -> 46.8 mm
- net GM4: track 31.3 -> 63.4 mm, vias 4 -> 5
- net ROW2: track 0.00 -> 26.8 mm, vias 0 -> 1
- net ROW1: track 0.00 -> 25.5 mm, vias 0 -> 1
- net GM2: track 21.6 -> 45.8 mm, vias 4 -> 5
- net ROW3: track 0.00 -> 24.2 mm, vias 0 -> 1
- net ROW0: track 0.00 -> 22.3 mm, vias 0 -> 1
- net GM1: track 26.1 -> 43.2 mm, vias 0 -> 1
- net GM_LAMP_POLARIZATION: track 85.8 -> 96.6 mm
- net COL1: track 65.9 -> 55.5 mm, vias 1 -> 0
- net COL0: track 59.9 -> 49.9 mm
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