File: hardware/Detector/chamber.kicad_pcb (KiCad board)
At the start: 2 copper layers, 89.9 x 82.6 mm, 121 parts, among them J1 USB_B_Micro, J10 Conn_02x02_Odd_Even, J11 Conn_02x02_Odd_Even, J12 Conn_02x02_Odd_Even, J13 Conn_02x02_Odd_Even, J14 Conn_02x02_Odd_Even, J15 Conn_02x02_Odd_Even, J16 Conn_02x02_Odd_Even, J17 Conn_02x02_Odd_Even, J2 Conn_02x02_Odd_Even, J3 Conn_02x02_Odd_Even, J4 Conn_02x02_Odd_Even, J5 Conn_02x02_Odd_Even, J51 Conn_02x05_Counter_Clockwise, J52 Conn_01x04, J6 Conn_02x02_Odd_Even, J7 Conn_02x02_Odd_Even, J8 Conn_02x02_Odd_Even, J9 Conn_02x02_Odd_Even, Q31 BC859, Q32 Q_NMOS_GDS, U1 STM32F030K6Tx, U2 HEF4093B, U31 MC34063AD

Commit message: backup
Parts:
- removed D42: LED, LED_SMD:LED_0603_1608Metric
- removed R19: 680R, Resistor_SMD:R_0805_2012Metric_Pad1.15x1.40mm_HandSolder
- added R36: 100k, Resistor_SMD:R_0805_2012Metric_Pad1.15x1.40mm_HandSolder, F.Cu at (174.0, 79.8)
- added TP1: TestPoint, TestPoint:TestPoint_Pad_D1.0mm, F.Cu at (169.4, 77.0)
- added TP2: TestPoint, TestPoint:TestPoint_Pad_D1.0mm, F.Cu at (169.4, 75.2)
- added TP3: TestPoint, TestPoint:TestPoint_Pad_D1.0mm, F.Cu at (160.8, 85.1)
- added TP4: TestPoint, TestPoint:TestPoint_Pad_D1.0mm, F.Cu at (160.8, 86.9)
- added TP5: TestPoint, TestPoint:TestPoint_Pad_D1.0mm, F.Cu at (173.7, 86.9)
- added TP6: TestPoint, TestPoint:TestPoint_Pad_D1.0mm, F.Cu at (160.3, 79.5)
- added TP7: TestPoint, TestPoint:TestPoint_Pad_D1.0mm, F.Cu at (160.5, 81.3)
- added TP8: TestPoint, TestPoint:TestPoint_Pad_D1.0mm, F.Cu at (158.8, 82.0)
- added TP9: TestPoint, TestPoint:TestPoint_Pad_D1.0mm, F.Cu at (163.1, 88.6)
- added U3: LCD_I2C, MuonDetector:LCD_I2C, F.Cu at (166.1, 100.6)
- moved J4 72.1 mm to (118.4, 78.2)
- moved J5 72.1 mm to (118.4, 78.2)
- moved R27 28.6 mm to (182.4, 93.5), turned to 0 degrees
- moved D51 21.6 mm to (154.2, 76.7)
- moved R59 19.9 mm to (165.1, 90.2)
- moved R60 19.3 mm to (168.7, 94.7)
- moved D40 16.8 mm to (143.0, 83.3)
- moved C1 16.5 mm to (147.8, 79.2)
- moved R30 16.4 mm to (182.6, 90.9), turned to 0 degrees
- moved H3 15.3 mm to (111.0, 74.2)
- moved H4 15.2 mm to (189.2, 74.2)
- moved R17 15.2 mm to (141.2, 81.0)
- moved J1 15.0 mm to (118.1, 70.1), turned to 180 degrees
- moved R29 14.4 mm to (150.1, 81.0)
- moved R18 10.8 mm to (147.8, 84.1)
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Connections:
- net /DataAcquisition/RST renamed /DataAcquisition/NRST
- D40 pad 2: (no net) -> Net-(D40-Pad2)
- D41 pad 2: (no net) -> Net-(D41-Pad2)
- J51 pad 10: (no net) -> /DataAcquisition/SWCLK
- J51 pad 9: (no net) -> /DataAcquisition/SWDIO
- J52 pad 1: (no net) -> VCC_5V
- J52 pad 2: (no net) -> /DataAcquisition/TX
- J52 pad 3: (no net) -> /DataAcquisition/RX
- R59 pad 1: (no net) -> Net-(R59-Pad1)
- R60 pad 1: (no net) -> Net-(R60-Pad1)
- U1 pad 10: (no net) -> Net-(TP7-Pad1)
- U1 pad 11: ROW3 -> Net-(TP8-Pad1)
- U1 pad 12: ROW2 -> ROW3
- U1 pad 13: ROW1 -> ROW2
- U1 pad 14: (no net) -> Net-(TP3-Pad1)
- U1 pad 15: (no net) -> Net-(TP4-Pad1)
- U1 pad 18: ROW0 -> Net-(TP9-Pad1)
- U1 pad 19: (no net) -> Net-(R59-Pad1)
- U1 pad 2: (no net) -> Net-(TP1-Pad1)
- U1 pad 20: (no net) -> Net-(R60-Pad1)
- U1 pad 21: COL0 -> ROW1
- U1 pad 22: COL1 -> ROW0
- U1 pad 23: COL2 -> /DataAcquisition/SWDIO
- U1 pad 24: COL3 -> /DataAcquisition/SWCLK
- U1 pad 25: (no net) -> Net-(TP5-Pad1)
- U1 pad 26: (no net) -> COL2
- U1 pad 27: (no net) -> COL3
- U1 pad 28: (no net) -> COL0
- U1 pad 29: (no net) -> /DataAcquisition/TX
- U1 pad 3: (no net) -> Net-(TP2-Pad1)
- U1 pad 30: (no net) -> /DataAcquisition/RX
- U1 pad 31: (no net) -> Net-(R36-Pad2)
- U1 pad 6: (no net) -> Net-(D41-Pad2)
- U1 pad 7: (no net) -> Net-(D40-Pad2)
- U1 pad 8: (no net) -> COL1
- U1 pad 9: (no net) -> Net-(TP6-Pad1)
Routing:
- net COL2: track 55.3 -> 132.4 mm, vias 4 -> 6
- net COL3: track 61.3 -> 136.6 mm, vias 0 -> 1
- net GM1: track 43.2 -> 71.9 mm, vias 1 -> 2
- net (no net): track 28.0 -> 0.00 mm, vias 0 -> 1
- net GM3: track 47.0 -> 67.8 mm, vias 1 -> 2
- net GM2: track 45.8 -> 64.5 mm, vias 5 -> 6
- net GND: track 17.9 -> 4.62 mm, vias 5 -> 6
- net Net-(R60-Pad1): track 0.00 -> 8.85 mm
- net VCC_5V: track 141.7 -> 132.9 mm, vias 2 -> 0
- net COL1: track 55.5 -> 47.8 mm
- net COL0: track 49.9 -> 42.2 mm
- net Net-(R59-Pad1): track 0.00 -> 6.45 mm
- net ROW2: track 26.8 -> 32.1 mm, vias 1 -> 2
- net Net-(TP2-Pad1): track 0.00 -> 4.66 mm
- net Net-(TP8-Pad1): track 0.00 -> 4.54 mm
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Other:
- board text added: "400V DC GM polarization"
- board text added: "CosmicRayDetector rev1.0"
- board text removed: "400V DC chamber polarization"
- board text removed: "Ionization Chamber Sensor rev4.0"

Commit message: roughly routed, to be polished
Parts:
- removed D51: 1n148, Diode_SMD:D_MiniMELF
- moved R28 34.4 mm to (182.4, 93.0), turned to 0 degrees
- moved R29 33.7 mm to (182.4, 90.9), turned to 0 degrees
- moved D41 33.1 mm to (165.6, 74.9), turned to 270 degrees
- moved R17 24.7 mm to (164.1, 71.6), turned to 270 degrees
- moved D40 22.7 mm to (164.1, 74.9), turned to 270 degrees
- moved R18 21.7 mm to (165.6, 71.6), turned to 270 degrees
- moved J52 20.6 mm to (181.4, 71.9)
- moved J1 19.6 mm to (137.7, 71.6)
- moved J51 13.0 mm to (161.5, 74.2)
- moved D1 12.1 mm to (138.4, 75.4)
- moved J4 7.33 mm to (124.5, 82.3), turned to 0 degrees
- moved J5 7.33 mm to (124.5, 82.3), turned to 0 degrees
- moved R1 6.89 mm to (133.6, 75.4), turned to 180 degrees
- moved C1 6.76 mm to (142.2, 75.4), turned to 180 degrees
- moved R30 2.05 mm to (182.4, 88.9)
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Connections:
- J51 pad 5: /DataAcquisition/VCC_PROG -> VCC_5V
- J51 pad 6: (no net) -> VCC_5V
- U1 pad 1: /DataAcquisition/VCC_PROG -> VCC_5V
- U1 pad 17: /DataAcquisition/VCC_PROG -> VCC_5V
- U1 pad 28: COL0 -> COL1
- U1 pad 5: /DataAcquisition/VCC_PROG -> VCC_5V
- U1 pad 8: COL1 -> COL0
Routing:
- net VCC_5V: track 132.9 -> 258.8 mm
- net /DataAcquisition/SWCLK: track 0.00 -> 35.9 mm, vias 0 -> 1
- net COL0: track 42.2 -> 70.2 mm, vias 4 -> 6
- net /DataAcquisition/SWDIO: track 0.00 -> 24.0 mm, vias 0 -> 1
- net COL1: track 47.8 -> 68.0 mm, vias 0 -> 2
- net /DataAcquisition/TX: track 0.00 -> 17.2 mm
- net /DataAcquisition/RX: track 0.00 -> 14.5 mm
- net /DataAcquisition/VCC_PROG: track 13.8 -> 0.00 mm
- net /DataAcquisition/NRST: track 0.00 -> 9.65 mm, vias 0 -> 1
- net GND: track 4.62 -> 10.9 mm
- net Net-(D40-Pad2): track 0.00 -> 3.96 mm
- net Net-(D41-Pad2): track 0.00 -> 3.66 mm
- net Net-(D1-Pad1): track 0.00 -> 2.86 mm
- net COL2: track 132.4 -> 134.6 mm, vias 6 -> 7
- net COL3: track 136.6 -> 138.8 mm, vias 1 -> 2
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
Commit message: before rename
Routing:
- net VCC_5V: track 258.8 -> 262.8 mm
- net Net-(TP7-Pad1): track 0.00 -> 2.70 mm
- net Net-(TP5-Pad1): track 0.00 -> 2.49 mm
- net GND: vias 6 -> 8
Changed lines of the file:
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@@
     (thickness 1.6)
     (drawings 13)
-    (tracks 715)
+    (tracks 731)
     (zones 0)
     (modules 129)
@@
   (segment (start 140.578 72.2805) (end 140.1305 72.728) (width 0.254) (layer F.Cu) (net 1))
   (segment (start 140.578 70.428) (end 140.578 72.2805) (width 0.254) (layer F.Cu) (net 1))
+  (via (at 167.386 72.644) (size 1) (drill 0.5) (layers F.Cu B.Cu) (net 1))
+  (via (at 167.132 70.866) (size 1) (drill 0.5) (layers F.Cu B.Cu) (net 1))
   (via (at 169.164 90.424) (size 1) (drill 0.5) (layers F.Cu B.Cu) (net 52))
   (segment (start 128.176 148.402) (end 128.125 148.453) (width 0.3048) (layer F.Cu) (net 2) (status 30))
@@
   (segment (start 138.968 75.0385) (end 139.3675 75.438) (width 0.254) (layer F.Cu) (net 10))
   (segment (start 138.968 73.088) (end 138.968 75.0385) (width 0.254) (layer F.Cu) (net 10))
-  (segment (start 166.774984 70.461016) (end 167.132 70.104) (width 0.254) (layer F.Cu) (net 10))
-  (segment (start 166.774984 78.075984) (end 166.774984 70.461016) (width 0.254) (layer F.Cu) (net 10))
-  (segment (start 166.986 78.287) (end 166.774984 78.075984) (width 0.254) (layer F.Cu) (net 10))
-  (segment (start 166.986 79.137) (end 166.986 78.287) (width 0.254) (layer F.Cu) (net 10))
   (segment (start 180.682 70.104) (end 167.132 70.104) (width 0.254) (layer F.Cu) (net 10))
   (segment (start 139.3675 75.438) (end 141.215 75.438) (width 0.254) (layer F.Cu) (net 10))
@@
   (segment (start 143.002 77.225) (end 153.407 77.225) (width 0.254) (layer F.Cu) (net 10))
   (segment (start 156.464 74.168) (end 156.464 71.628) (width 0.254) (layer F.Cu) (net 10))
-  (segment (start 166.68901 70.104) (end 167.132 70.104) (width 0.254) (layer F.Cu) (net 10))
-  (segment (start 166.319376 69.64699) (end 166.68901 70.016624) (width 0.254) (layer F.Cu) (net 10))
+  (segment (start 191.128 83.618) (end 189.806 82.296) (width 0.254) (layer B.Cu) (net 10))
+  (segment (start 191.128 84.372) (end 191.128 83.618) (width 0.254) (layer B.Cu) (net 10))
+  (segment (start 183.397 90.932) (end 183.397 88.9) (width 0.254) (layer F.Cu) (net 10))
+  (segment (start 183.397 94.996) (end 183.397 92.964) (width 0.254) (layer F.Cu) (net 10))
+  (segment (start 166.68901 70.016624) (end 166.68901 69.66101) (width 0.254) (layer F.Cu) (net 10))
   (segment (start 164.896624 69.64699) (end 166.319376 69.64699) (width 0.254) (layer F.Cu) (net 10))
-  (segment (start 164.8415 69.702114) (end 164.896624 69.64699) (width 0.254) (layer F.Cu) (net 10))
+  (segment (start 164.795376 69.65599) (end 164.8415 69.702114) (width 0.254) (layer F.Cu) (net 10))
   (segment (start 163.372624 69.65599) (end 164.795376 69.65599) (width 0.254) (layer F.Cu) (net 10))
+  (segment (start 166.68901 69.66101) (end 167.132 70.104) (width 0.254) (layer F.Cu) (net 10))
+  (segment (start 157.313999 70.778001) (end 157.313999 70.270001) (width 0.254) (layer F.Cu) (net 10))
   (segment (start 156.464 71.628) (end 157.313999 70.778001) (width 0.254) (layer F.Cu) (net 10))
+  (segment (start 166.319376 69.64699) (end 166.68901 70.016624) (width 0.254) (layer F.Cu) (net 10))
   (segment (start 157.313999 70.270001) (end 158.242 69.342) (width 0.254) (layer F.Cu) (net 10))
-  (segment (start 157.313999 70.778001) (end 157.313999 70.270001) (width 0.254) (layer F.Cu) (net 10))
   (segment (start 158.242 69.342) (end 163.00299 69.342) (width 0.254) (layer F.Cu) (net 10))
-  (segment (start 166.68901 70.016624) (end 166.68901 70.104) (width 0.254) (layer F.Cu) (net 10))
   (segment (start 163.00299 69.342) (end 163.00299 70.025624) (width 0.254) (layer F.Cu) (net 10))
-  (segment (start 164.795376 69.65599) (end 164.8415 69.702114) (width 0.254) (layer F.Cu) (net 10))
+  (segment (start 164.8415 69.702114) (end 164.896624 69.64699) (width 0.254) (layer F.Cu) (net 10))
   (segment (start 163.00299 70.025624) (end 163.372624 69.65599) (width 0.254) (layer F.Cu) (net 10))
-  (segment (start 191.128 83.618) (end 189.806 82.296) (width 0.254) (layer B.Cu) (net 10))
-  (segment (start 191.128 84.372) (end 191.128 83.618) (width 0.254) (layer B.Cu) (net 10))
-  (segment (start 183.397 90.932) (end 183.397 88.9) (width 0.254) (layer F.Cu) (net 10))
-  (segment (start 183.397 94.996) (end 183.397 92.964) (width 0.254) (layer F.Cu) (net 10))
+  (segment (start 168.402 70.104) (end 167.132 70.104) (width 0.254) (layer F.Cu) (net 10))
+  (segment (start 168.304772 76.05291) (end 168.402 75.955682) (width 0.254) (layer F.Cu) (net 10))
+  (segment (start 167.910403 75.65854) (end 168.304772 76.05291) (width 0.254) (layer F.Cu) (net 10))
+  (segment (start 167.064641 75.65854) (end 167.910403 75.65854) (width 0.254) (layer F.Cu) (net 10))
+  (segment (start 166.606521 76.11666) (end 167.064641 75.65854) (width 0.254) (layer F.Cu) (net 10))
+  (segment (start 166.986 78.287) (end 167.27799 77.99501) (width 0.254) (layer F.Cu) (net 10))
+  (segment (start 168.402 75.955682) (end 168.402 70.104) (width 0.254) (layer F.Cu) (net 10))
+  (segment (start 166.986 79.137) (end 166.986 78.287) (width 0.254) (layer F.Cu) (net 10))
+  (segment (start 167.27799 77.99501) (end 167.27799 77.420542) (width 0.254) (layer F.Cu) (net 10))
+  (segment (start 167.27799 77.420542) (end 167.064641 77.420542) (width 0.254) (layer F.Cu) (net 10))
+  (segment (start 167.064641 77.420542) (end 166.606521 76.962422) (width 0.254) (layer F.Cu) (net 10))
+  (segment (start 166.606521 76.962422) (end 166.606521 76.11666) (width 0.254) (layer F.Cu) (net 10))
   (segment (start 190.84 137.595) (end 190.84 131.595) (width 0.3048) (layer F.Cu) (net 11))
   (segment (start 186.112 137.595) (end 185.492 136.975) (width 0.3048) (layer F.Cu) (net 11))
@@
   (segment (start 156.46399 79.24799) (end 161.568052 79.24799) (width 0.254) (layer B.Cu) (net 57))
   (segment (start 151.384 74.168) (end 156.46399 79.24799) (width 0.254) (layer B.Cu) (net 57))
-  (via (at 167.655985 76.708) (size 1) (drill 0.5) (layers F.Cu B.Cu) (net 58))
-  (segment (start 165.115985 74.168) (end 167.155986 76.208001) (width 0.254) (layer B.Cu) (net 58))
-  (segment (start 167.155986 76.208001) (end 167.655985 76.708) (width 0.254) (layer B.Cu) (net 58))
+  (segment (start 167.655981 76.708) (end 167.487522 76.539541) (width 0.254) (layer B.Cu) (net 58))
+  (segment (start 167.786 79.137) (end 167.786 76.838019) (width 0.254) (layer F.Cu) (net 58))
+  (via (at 167.487522 76.539541) (size 1) (drill 0.5) (layers F.Cu B.Cu) (net 58))
+  (segment (start 167.786 76.838019) (end 167.487522 76.539541) (width 0.254) (layer F.Cu) (net 58))
   (segment (start 161.544 74.168) (end 165.115985 74.168) (width 0.254) (layer B.Cu) (net 58))
-  (segment (start 167.786 76.838015) (end 167.655985 76.708) (width 0.254) (layer F.Cu) (net 58))
-  (segment (start 167.786 79.137) (end 167.786 76.838015) (width 0.254) (layer F.Cu) (net 58))
+  (segment (start 165.115985 74.168) (end 167.655985 76.708) (width 0.254) (layer B.Cu) (net 58))
+  (segment (start 167.655985 76.708) (end 167.655981 76.708) (width 0.254) (layer B.Cu) (net 58))
   (segment (start 167.386 92.484) (end 167.386 90.424) (width 0.254) (layer F.Cu) (net 59))
   (segment (start 166.186 89.224) (end 166.186 87.487) (width 0.254) (layer F.Cu) (net 59))
@@
   (segment (start 169.386 76.994) (end 169.418 76.962) (width 0.254) (layer F.Cu) (net 61))
   (segment (start 169.386 79.137) (end 169.386 76.994) (width 0.254) (layer F.Cu) (net 61))
-  (segment (start 168.586 79.137) (end 168.586 78.287) (width 0.254) (layer F.Cu) (net 62))
+  (segment (start 168.536999 78.237999) (end 168.536999 76.539119) (width 0.254) (layer F.Cu) (net 62))
   (segment (start 168.586 78.287) (end 168.536999 78.237999) (width 0.254) (layer F.Cu) (net 62))
-  (segment (start 168.536999 78.237999) (end 168.536999 76.065001) (width 0.254) (layer F.Cu) (net 62))
-  (segment (start 168.536999 76.065001) (end 168.918001 75.683999) (width 0.254) (layer F.Cu) (net 62))
+  (segment (start 168.536999 76.539119) (end 168.918001 76.158117) (width 0.254) (layer F.Cu) (net 62))
   (segment (start 168.918001 75.683999) (end 169.418 75.184) (width 0.254) (layer F.Cu) (net 62))
+  (segment (start 168.586 79.137) (end 168.586 78.287) (width 0.254) (layer F.Cu) (net 62))
+  (segment (start 168.918001 76.158117) (end 168.918001 75.683999) (width 0.254) (layer F.Cu) (net 62))
   (segment (start 161.36 84.512) (end 160.782 85.09) (width 0.254) (layer F.Cu) (net 63))
   (segment (start 163.211 84.512) (end 161.36 84.512) (width 0.254) (layer F.Cu) (net 63))
   (segment (start 162.338 85.312) (end 163.211 85.312) (width 0.254) (layer F.Cu) (net 64))
   (segment (start 160.782 86.868) (end 162.338 85.312) (width 0.254) (layer F.Cu) (net 64))
+  (segment (start 172.317 86.868) (end 171.561 86.112) (width 0.254) (layer F.Cu) (net 65))
+  (segment (start 173.736 86.868) (end 172.317 86.868) (width 0.254) (layer F.Cu) (net 65))
   (segment (start 162.201 79.502) (end 160.274 79.502) (width 0.254) (layer F.Cu) (net 66))
   (segment (start 163.211 80.512) (end 162.201 79.502) (width 0.254) (layer F.Cu) (net 66))
+  (segment (start 160.56 81.312) (end 160.528 81.28) (width 0.254) (layer F.Cu) (net 67))
+  (segment (start 163.211 81.312) (end 160.56 81.312) (width 0.254) (layer F.Cu) (net 67))
   (segment (start 159.457106 82.042) (end 158.75 82.042) (width 0.254) (layer F.Cu) (net 68))
   (segment (start 159.592105 82.176999) (end 159.457106 82.042) (width 0.254) (layer F.Cu) (net 68))
