File: hardware/FPGABoardMockup/FPGABoardMockup.kicad_pcb (KiCad board)
At the start: 2 copper layers, 104 x 66 mm, 16 parts, among them J1 Conn_02x14_Odd_Even, J2 Conn_02x11_Counter_Clockwise, J3 Barrel_Jack, J4 Conn_02x05_Counter_Clockwise, J5 USB_B_Mini, J6 Conn_02x05_Counter_Clockwise, J7 Conn_02x14_Odd_Even, J8 Conn_02x11_Counter_Clockwise, SW1 SW_Push, SW2 SW_Push, SW3 SW_Push, SW4 SW_Push

Commit message: fix #55
Parts:
- SW1, SW3, SW4: footprint Button_Switch_SMD:SW_SPST_B3U-1000P-B -> Button_Switch_SMD:SW_SPST_CK_RS282G05A3
- SW2: footprint Button_Switch_SMD:SW_SPST_PTS645 -> Button_Switch_SMD:SW_SPST_CK_RS282G05A3
- moved J3 12.0 mm to (114.0, 100.0), turned to 270 degrees
